Commit message: change to prefix only in urdfs

File: mir_description/urdf/include/mir_100.gazebo.xacro (robot description, xacro)
@@ -2,10 +2,10 @@
 <robot xmlns:xacro="http://ros.org/wiki/xacro">
   <!-- See https://github.com/ros-simulation/gazebo_ros_pkgs/wiki/ROS-2-Migration:-Diff-drive for ros2 information -->
-  <xacro:macro name="diff_controller_plugin_gazebo" params="prefix namespace left_wheel_joint right_wheel_joint wheel_separation wheel_radius">
+  <xacro:macro name="diff_controller_plugin_gazebo" params="prefix left_wheel_joint right_wheel_joint wheel_separation wheel_radius">
     <gazebo>
       <!-- Use gazebo_ros_joint_state_publisher instead of publishWheelJointState -->
       <plugin name="joint_states" filename="libgazebo_ros_joint_state_publisher.so">
         <ros>
-          <namespace>${namespace}</namespace>
+          <namespace>${prefix}</namespace>
         </ros>
         <update_rate>1000.0</update_rate>
@@ -52,9 +52,9 @@
   </xacro:macro>
  <!-- See https://github.com/ros-simulation/gazebo_ros_pkgs/wiki/ROS-2-Migration:-P3D for ros2 information -->
-  <xacro:macro name="p3d_base_controller" params="namespace prefix">
+  <xacro:macro name="p3d_base_controller" params="prefix">
     <gazebo>
       <plugin name="p3d_base_controller" filename="libgazebo_ros_p3d.so">
         <ros>
-          <namespace>${namespace}</namespace>
+          <namespace>${prefix}</namespace>
           <remapping>odom:=base_pose_ground_truth</remapping>
         </ros>

File: mir_description/urdf/include/mir_100_v1.urdf.xacro (robot description, xacro)
@@ -24,5 +24,5 @@
   <xacro:property name="mir_100_caster_wheel_base_dz" value="${mir_100_caster_wheel_radius-mir_100_caster_wheel_dz}" />
   <xacro:property name="imu_stdev" value="0.00017" />
-  <xacro:macro name="actuated_wheel" params="prefix namespace locationprefix locationright">
+  <xacro:macro name="actuated_wheel" params="prefix  locationprefix locationright">
     <joint name="${prefix}${locationprefix}_wheel_joint" type="continuous">
       <origin xyz="0.0 ${-mir_100_act_wheel_dy * locationright} ${mir_100_act_wheel_radius}" rpy="0 0 0" />
@@ -111,5 +111,5 @@
       <plugin name="${locationprefix}_caster_wheel_joint_states" filename="libgazebo_ros_joint_state_publisher.so">
         <ros>
-          <namespace>${namespace}</namespace>
+          <namespace>${prefix}</namespace>
         </ros>
         <update_rate>200.0</update_rate>
@@ -139,5 +139,5 @@
     </gazebo>
   </xacro:macro>
-  <xacro:macro name="mir_100" params="prefix namespace">
+  <xacro:macro name="mir_100" params="prefix">
     <link name="${prefix}base_footprint" />
     <joint name="${prefix}base_joint" type="fixed">
@@ -198,5 +198,5 @@
       <origin xyz="0.4288 0.2358 0.1914" rpy="0.0 0.0 ${0.25 * pi}" />  <!-- from visually matching up the meshes of the MiR and the laser scanner -->
     </joint>
-    <xacro:sick_s300 prefix="${prefix}" namespace="${namespace}" link="front_laser_link" topic="f_scan" />
+    <xacro:sick_s300 prefix="${prefix}" link="front_laser_link" topic="f_scan" />
     <joint name="${prefix}base_link_to_back_laser_joint" type="fixed">
       <parent link="${prefix}base_link" />
@@ -204,5 +204,5 @@
       <origin xyz="-0.3548 -0.2352 0.1914" rpy="0.0 0.0 ${-0.75 * pi}" />  <!-- from visually matching up the meshes of the MiR and the laser scanner -->
     </joint>
-    <xacro:sick_s300 prefix="${prefix}" namespace="${namespace}" link="back_laser_link" topic="b_scan" />
+    <xacro:sick_s300 prefix="${prefix}" link="back_laser_link" topic="b_scan" />
     <!-- Ultrasound sensors -->
     <joint name="${prefix}us_1_joint" type="fixed">   <!-- right ultrasound -->
@@ -219,6 +219,6 @@
     <link name="${prefix}us_2_frame" />
     <!-- wheels -->
-    <xacro:actuated_wheel prefix="${prefix}" namespace="${namespace}" locationprefix="left" locationright="-1"/>
-    <xacro:actuated_wheel prefix="${prefix}" namespace="${namespace}" locationprefix="right" locationright="1"/>
+    <xacro:actuated_wheel prefix="${prefix}" locationprefix="left" locationright="-1"/>
+    <xacro:actuated_wheel prefix="${prefix}" locationprefix="right" locationright="1"/>
     <xacro:caster_wheel prefix="${prefix}" locationprefix="fl" locationright="-1" wheel_base_dx="${mir_100_front_caster_wheel_base_dx}"/>
     <xacro:caster_wheel prefix="${prefix}" locationprefix="fr" locationright="1" wheel_base_dx="${mir_100_front_caster_wheel_base_dx}"/>
@@ -235,5 +235,5 @@
     <!-- set the gazebo friction parameters for the wheels -->
     <xacro:set_all_wheel_frictions prefix="${prefix}"/>
-    <xacro:p3d_base_controller prefix="${prefix}" namespace="${namespace}"/>
+    <xacro:p3d_base_controller prefix="${prefix}"/>
   </xacro:macro>
 </robot>

File: mir_description/urdf/include/sick_s300.urdf.xacro (robot description, xacro)
@@ -6,5 +6,5 @@
   <xacro:property name="laser_z" value="0.185" />
   <xacro:property name="laser_mass" value="2.0" />
-  <xacro:macro name="sick_s300" params="link topic prefix namespace">
+  <xacro:macro name="sick_s300" params="link topic prefix">
     <link name="${prefix}${link}">
       <visual>
@@ -58,5 +58,5 @@
           <ros>
             <remapping>~/out:=${topic}</remapping>
-            <namespace>${namespace}</namespace>
+            <namespace>${prefix}</namespace>
           </ros>
           <output_type>sensor_msgs/LaserScan</output_type>

File: mir_description/urdf/mir.urdf.xacro (robot description, xacro)
@@ -5,20 +5,17 @@
   <xacro:include filename="$(find mir_description)/urdf/include/mir_100_v1.urdf.xacro" />
   <xacro:include filename="$(find mir_description)/urdf/include/common.gazebo.xacro" />
-  <xacro:arg name="namespace" default=""/>
   <xacro:arg name="tf_prefix" default="" />
   <xacro:property name="tf_prefix_val" value="$(arg tf_prefix)" />
   <xacro:if value="${tf_prefix_val == ''}">
     <xacro:property name="prefix" value="" />
-    <xacro:property name="namespace" value=""/>
   </xacro:if>
   <xacro:unless value="${tf_prefix_val == ''}">
     <xacro:property name="prefix" value="${tf_prefix_val}/" />
-    <xacro:property name="namespace" value="${tf_prefix_val}"/>
   </xacro:unless>
-  <xacro:mir_100 prefix="${prefix}" namespace="${namespace}"/>
+  <xacro:mir_100 prefix="${prefix}"/>
   <!--
   <xacro:controller_plugin_gazebo robot_namespace=""/>
   -->
-  <xacro:diff_controller_plugin_gazebo prefix="${prefix}" namespace="${namespace}"
+  <xacro:diff_controller_plugin_gazebo prefix="${prefix}"
     left_wheel_joint="${prefix}left_wheel_joint"
     right_wheel_joint="${prefix}right_wheel_joint"

Commit message: resolved gazeboplugin namespace errors

File: mir_description/urdf/include/mir_100.gazebo.xacro (robot description, xacro)
@@ -2,10 +2,10 @@
 <robot xmlns:xacro="http://ros.org/wiki/xacro">
   <!-- See https://github.com/ros-simulation/gazebo_ros_pkgs/wiki/ROS-2-Migration:-Diff-drive for ros2 information -->
-  <xacro:macro name="diff_controller_plugin_gazebo" params="prefix left_wheel_joint right_wheel_joint wheel_separation wheel_radius">
+  <xacro:macro name="diff_controller_plugin_gazebo" params="prefix ns left_wheel_joint right_wheel_joint wheel_separation wheel_radius">
     <gazebo>
       <!-- Use gazebo_ros_joint_state_publisher instead of publishWheelJointState -->
       <plugin name="joint_states" filename="libgazebo_ros_joint_state_publisher.so">
         <ros>
-          <remapping>joint_states:=${prefix}joint_states_demo</remapping>
+          <namespace>${ns}</namespace>
         </ros>
         <update_rate>1000.0</update_rate>

File: mir_description/urdf/include/mir_100_v1.urdf.xacro (robot description, xacro)
@@ -54,5 +54,5 @@
     </gazebo>
   </xacro:macro>
-  <xacro:macro name="caster_wheel" params="prefix locationprefix locationright wheel_base_dx">
+  <xacro:macro name="caster_wheel" params="prefix ns locationprefix locationright wheel_base_dx">
     <!-- caster hub -->
     <joint name="${prefix}${locationprefix}_caster_rotation_joint" type="continuous">
@@ -66,4 +66,5 @@
       <plugin name="${locationprefix}_caster_rotation_joint_states" filename="libgazebo_ros_joint_state_publisher.so">
         <ros>
+          <namespace>${ns}</namespace>
         </ros>
         <update_rate>200.0</update_rate>
@@ -111,5 +112,5 @@
       <plugin name="${locationprefix}_caster_wheel_joint_states" filename="libgazebo_ros_joint_state_publisher.so">
         <ros>
-          <remapping>joint_states:=${prefix}joint_states_demo</remapping>
+          <namespace>${ns}</namespace>
         </ros>
         <update_rate>200.0</update_rate>
@@ -139,5 +140,5 @@
     </gazebo>
   </xacro:macro>
-  <xacro:macro name="mir_100" params="prefix">
+  <xacro:macro name="mir_100" params="prefix ns">
     <link name="${prefix}base_footprint" />
     <joint name="${prefix}base_joint" type="fixed">
@@ -221,8 +222,8 @@
     <xacro:actuated_wheel prefix="${prefix}" locationprefix="left" locationright="-1"/>
     <xacro:actuated_wheel prefix="${prefix}" locationprefix="right" locationright="1"/>
-    <xacro:caster_wheel prefix="${prefix}" locationprefix="fl" locationright="-1" wheel_base_dx="${mir_100_front_caster_wheel_base_dx}"/>
-    <xacro:caster_wheel prefix="${prefix}" locationprefix="fr" locationright="1" wheel_base_dx="${mir_100_front_caster_wheel_base_dx}"/>
-    <xacro:caster_wheel prefix="${prefix}" locationprefix="bl" locationright="-1" wheel_base_dx="${mir_100_back_caster_wheel_base_dx}"/>
-    <xacro:caster_wheel prefix="${prefix}" locationprefix="br" locationright="1" wheel_base_dx="${mir_100_back_caster_wheel_base_dx}"/>
+    <xacro:caster_wheel prefix="${prefix}" ns="${ns}" locationprefix="fl" locationright="-1" wheel_base_dx="${mir_100_front_caster_wheel_base_dx}"/>
+    <xacro:caster_wheel prefix="${prefix}" ns="${ns}" locationprefix="fr" locationright="1" wheel_base_dx="${mir_100_front_caster_wheel_base_dx}"/>
+    <xacro:caster_wheel prefix="${prefix}" ns="${ns}" locationprefix="bl" locationright="-1" wheel_base_dx="${mir_100_back_caster_wheel_base_dx}"/>
+    <xacro:caster_wheel prefix="${prefix}" ns="${ns}" locationprefix="br" locationright="1" wheel_base_dx="${mir_100_back_caster_wheel_base_dx}"/>
     <joint name="${prefix}base_link_surface_joint" type="fixed">
       <origin xyz="${mir_100_act_wheel_dx} 0 0.352" rpy="0 0 0" />

File: mir_description/urdf/mir.urdf.xacro (robot description, xacro)
@@ -5,17 +5,15 @@
   <xacro:include filename="$(find mir_description)/urdf/include/mir_100_v1.urdf.xacro" />
   <xacro:include filename="$(find mir_description)/urdf/include/common.gazebo.xacro" />
+  <xacro:include filename="$(find mir_description)/urdf/include/mir_100.gazebo.xacro" />
   <xacro:arg name="tf_prefix" default="" />
-  <xacro:property name="tf_prefix_val" value="$(arg tf_prefix)" />
-  <xacro:if value="${tf_prefix_val == ''}">
+  <xacro:property name="ns" value="$(arg tf_prefix)" />
+  <xacro:if value="${ns == ''}">
     <xacro:property name="prefix" value="" />
   </xacro:if>
-  <xacro:unless value="${tf_prefix_val == ''}">
-    <xacro:property name="prefix" value="${tf_prefix_val}/" />
+  <xacro:unless value="${ns == ''}">
+    <xacro:property name="prefix" value="${ns}/" />
   </xacro:unless>
-  <xacro:mir_100 prefix="${prefix}"/>
-  <!--
-  <xacro:controller_plugin_gazebo robot_namespace=""/>
-  -->
-  <xacro:diff_controller_plugin_gazebo prefix="${prefix}"
+  <xacro:mir_100 prefix="${prefix}" ns="${ns}"/>
+  <xacro:diff_controller_plugin_gazebo prefix="${prefix}" ns="${ns}"
     left_wheel_joint="${prefix}left_wheel_joint"
     right_wheel_joint="${prefix}right_wheel_joint"
