Commit message: separated wheel parts to simplify urdf build

File: mir_description/urdf/include/mir_100_v1.urdf.xacro (robot description, xacro)
@@ -6,4 +6,6 @@
   <xacro:include filename="$(find mir_description)/urdf/include/mir_100.transmission.xacro" />
   <xacro:include filename="$(find mir_description)/urdf/include/sick_s300.urdf.xacro" />
+  <xacro:include filename="$(find mir_description)/urdf/include/wheel.urdf.xacro" />
+  <xacro:include filename="$(find mir_description)/urdf/include/caster.urdf.xacro" />
   <xacro:property name="deg_to_rad" value="0.017453293" />
   <xacro:property name="mir_100_base_mass" value="58.0" />
@@ -24,120 +26,4 @@
   <xacro:property name="mir_100_caster_wheel_base_dz" value="${mir_100_caster_wheel_radius-mir_100_caster_wheel_dz}" />
   <xacro:property name="imu_stdev" value="0.00017" />
-  <xacro:macro name="actuated_wheel" params="prefix  locationprefix locationright">
-    <joint name="${prefix}${locationprefix}_wheel_joint" type="continuous">
-      <origin xyz="0.0 ${-mir_100_act_wheel_dy * locationright} ${mir_100_act_wheel_radius}" rpy="0 0 0" />
-      <parent link="${prefix}base_link" />
-      <child link="${prefix}${locationprefix}_wheel_link" />
-      <axis xyz="0 1 0" />
-      <limit effort="100" velocity="20.0" />
-    </joint>
-    <link name="${prefix}${locationprefix}_wheel_link">
-      <xacro:cylinder_inertial mass="${mir_100_act_wheel_mass}" radius="${mir_100_act_wheel_radius}" length="${mir_100_act_wheel_width}">
-        <origin xyz="0 0 0" rpy="${0.5 * pi} 0 0" />
-      </xacro:cylinder_inertial>
-      <visual>
-        <origin xyz="0 0 0" rpy="0 0 0" />
-        <geometry>
-          <mesh filename="package://mir_description/meshes/visual/wheel.stl" />
-        </geometry>
-        <xacro:insert_block name="material_dark_grey" />
-      </visual>
-      <collision>
-        <origin xyz="0 0 0" rpy="${pi/2} 0 0" />
-        <geometry>
-          <cylinder radius="${mir_100_act_wheel_radius}" length="${mir_100_act_wheel_width}" />
-        </geometry>
-      </collision>
-    </link>
-    <gazebo reference="${prefix}${locationprefix}_wheel_link">
-      <material>Gazebo/DarkGrey</material>
-    </gazebo>
-  </xacro:macro>
-  <xacro:macro name="caster_wheel" params="prefix ns locationprefix locationright wheel_base_dx">
-    <!-- caster hub -->
-    <joint name="${prefix}${locationprefix}_caster_rotation_joint" type="continuous">
-      <origin xyz="${wheel_base_dx} ${-mir_100_caster_wheel_base_dy * locationright} ${mir_100_caster_wheel_base_dz}" rpy="0 0 0" />
-      <parent link="${prefix}base_link" />
-      <child link="${prefix}${locationprefix}_caster_rotation_link" />
-      <axis xyz="0 0 1" />
-      <dynamics damping="0.01" friction="0.0"/>
-    </joint>
-    <gazebo>
-      <plugin name="${locationprefix}_caster_rotation_joint_states" filename="libgazebo_ros_joint_state_publisher.so">
-        <ros>
-          <namespace>${ns}</namespace>
-        </ros>
-        <update_rate>200.0</update_rate>
-        <joint_name>${prefix}${locationprefix}_caster_rotation_joint</joint_name>
-      </plugin>
-    </gazebo>
-    <link name="${prefix}${locationprefix}_caster_rotation_link">
-      <inertial>
-        <!-- <origin xyz="0 0 -0.042500000044" rpy="${0.5 * pi} ${24 * deg_to_rad} ${1.5 * pi}" /> -->
-        <origin xyz="0 0 -0.042500000044" rpy="${24 * deg_to_rad} 0 ${0.5 * pi} " />
-        <mass value="0.3097539019" />
-        <inertia
-          ixx="0.0005844517978"
-          ixy="0"
-          ixz="0"
-          iyy="0.00052872551237"
-          iyz="0"
-          izz="0.00017923555074" />
-      </inertial>
-      <visual>
-        <origin xyz="0 0 0" rpy="0 0 0" />
-        <geometry>
-          <mesh filename="package://mir_description/meshes/visual/caster_wheel_base.stl" />
-        </geometry>
-        <xacro:insert_block name="material_silver" />
-      </visual>
-      <collision>
-        <origin xyz="0 0 0" rpy="0 0 0" />
-        <geometry>
-          <mesh filename="package://mir_description/meshes/collision/caster_wheel_base.stl" />
-        </geometry>
-      </collision>
-    </link>
-    <gazebo reference="${prefix}${locationprefix}_caster_rotation_link">
-      <material>Gazebo/Grey</material>
-    </gazebo>
-    <!-- caster wheel -->
-    <joint name="${prefix}${locationprefix}_caster_wheel_joint" type="continuous">
-      <origin xyz="${mir_100_caster_wheel_dx} ${-mir_100_caster_wheel_dy * locationright} ${mir_100_caster_wheel_dz}" rpy="0 0 0" />
-      <parent link="${prefix}${locationprefix}_caster_rotation_link" />
-      <child link="${prefix}${locationprefix}_caster_wheel_link" />
-      <axis xyz="0 1 0" />
-    </joint>
-    <gazebo>
-      <plugin name="${locationprefix}_caster_wheel_joint_states" filename="libgazebo_ros_joint_state_publisher.so">
-        <ros>
-          <namespace>${ns}</namespace>
-        </ros>
-        <update_rate>200.0</update_rate>
-        <joint_name>${prefix}${locationprefix}_caster_wheel_joint</joint_name>
-      </plugin>
-    </gazebo>
-    <link name="${prefix}${locationprefix}_caster_wheel_link">
-      <xacro:cylinder_inertial mass="${mir_100_caster_wheel_mass}" radius="${mir_100_caster_wheel_radius}" length="${mir_100_caster_wheel_width}">
-        <origin xyz="0 0 0" rpy="${0.5 * pi} 0 0" />
-      </xacro:cylinder_inertial>
-      <visual>
-        <origin xyz="0 0 0" rpy="0 0 0" />
-        <geometry>
-          <mesh filename="package://mir_description/meshes/visual/wheel.stl" />
-        </geometry>
-        <xacro:insert_block name="material_dark_grey" />
-      </visual>
-      <collision>
-        <origin xyz="0 0 0" rpy="${pi/2} 0 0" />
-        <geometry>
-          <cylinder radius="${mir_100_caster_wheel_radius}" length="${mir_100_caster_wheel_width}" />
-        </geometry>
-      </collision>
-    </link>
-    <gazebo reference="${prefix}${locationprefix}_caster_wheel_link">
-      <material>Gazebo/DarkGrey</material>
-    </gazebo>
-  </xacro:macro>
   <xacro:macro name="mir_100" params="prefix ns">
     <link name="${prefix}base_footprint" />
@@ -234,6 +120,4 @@
     <link name="${prefix}surface"/>
     <xacro:mir_100_wheel_transmissions prefix="${prefix}"/>
-    <!-- set the gazebo friction parameters for the wheels -->
-    <xacro:set_all_wheel_frictions prefix="${prefix}"/>
     <xacro:p3d_base_controller prefix="${prefix}"/>
   </xacro:macro>

Commit message: Changed MiR100 mass to 78.2kg

File: mir_description/urdf/include/mir_100_v1.urdf.xacro (robot description, xacro)
@@ -9,5 +9,4 @@
   <xacro:include filename="$(find mir_description)/urdf/include/caster.urdf.xacro" />
   <xacro:property name="deg_to_rad" value="0.017453293" />
-  <xacro:property name="mir_100_base_mass" value="58.0" />
   <xacro:property name="mir_100_act_wheel_radius" value="0.0625" />
   <xacro:property name="mir_100_act_wheel_width" value="0.032" />
@@ -25,4 +24,9 @@
   <xacro:property name="mir_100_caster_wheel_base_dy" value="0.203" />
   <xacro:property name="mir_100_caster_wheel_base_dz" value="${mir_100_caster_wheel_radius-mir_100_caster_wheel_dz}" />
+  <!-- MiR 100 complete mass 78.2kg (8.2kg battery) -->
+  <!-- - 2x2kg sick laser = 4kg-->
+  <!-- - 4x caster wheels + rotation link: 4x 1.31 kg -->
+  <!-- - 2x act wheels: 2kg -->
+  <xacro:property name="mir_100_base_mass" value="66.96" />
   <xacro:property name="imu_stdev" value="0.00017" />
   <xacro:macro name="mir_100" params="prefix ns">

Commit message: cherry-picked intertia from 91952d8

File: mir_description/urdf/include/mir_100_v1.urdf.xacro (robot description, xacro)
@@ -9,4 +9,13 @@
   <xacro:include filename="$(find mir_description)/urdf/include/caster.urdf.xacro" />
   <xacro:property name="deg_to_rad" value="0.017453293" />
+  <!-- The inertia for the MiR platform is intentionally chosen to be smaller than
+       the bounding box and also shifted a bit to the back, because most of the mass
+       is in the lower center back (because of the batteries). -->
+  <xacro:property name="mir_base_inertial_x" value="-0.05" />
+  <xacro:property name="mir_base_inertial_y" value="0.0" />
+  <xacro:property name="mir_base_inertial_z" value="0.15" />
+  <xacro:property name="mir_base_inertial_x_length" value="0.50" />
+  <xacro:property name="mir_base_inertial_y_length" value="0.30" />
+  <xacro:property name="mir_base_inertial_z_length" value="0.20" />
   <xacro:property name="mir_100_act_wheel_radius" value="0.0625" />
   <xacro:property name="mir_100_act_wheel_width" value="0.032" />
@@ -38,6 +47,6 @@
     </joint>
     <link name="${prefix}base_link">
-      <xacro:box_inertial mass="${mir_100_base_mass}" x="0.9" y="0.58" z="0.3">
-        <origin xyz="${mir_100_act_wheel_dx} 0 0.20" rpy="0 0 0" />
+      <xacro:box_inertial mass="${mir_100_base_mass}" x="${mir_base_inertial_x_length}" y="${mir_base_inertial_y_length}" z="${mir_base_inertial_z_length}">
+        <origin xyz="${mir_base_inertial_x + mir_100_act_wheel_dx} ${mir_base_inertial_y} ${mir_base_inertial_z}" rpy="0 0 0" />
       </xacro:box_inertial>
       <visual>
