Commit message: allow urdf to parse collision parameters for gazbeo

File: mir_description/urdf/include/caster.urdf.xacro (robot description, xacro)
@@ -92,10 +92,32 @@
     <!-- set the gazebo friction parameters for the wheels -->
     <gazebo reference="${prefix}${locationprefix}_caster_wheel_link">
-      <kp value="10000000.0"/>
-      <kd value="1.0"/>
-      <mu1 value="1"/>
-      <mu2 value="1"/>
-      <maxVel>1.0</maxVel>
-      <minDepth>0.01</minDepth>
+      <collision name="${prefix}${locationprefix}_caster_wheel_link_collision">
+        <surface>
+            <friction>
+              <ode>
+                <mu>1.0</mu>
+                <mu2>1.0</mu2>
+                <!--<fdir1>0 0 1</fdir1> -->
+                <!-- <slip1>0</slip1>
+                <slip2>0</slip2> -->
+              </ode>
+              <!-- <torsional>
+                <coefficient>200</coefficient>
+                <use_patch_radius>true</use_patch_radius>
+                <surface_radius>${mir_100_caster_wheel_radius}</surface_radius>
+              </torsional> -->
+            </friction>
+            <contact>
+              <ode>
+                <!-- <soft_cfm>0.0</soft_cfm>
+                <soft_erp>0.2</soft_erp> -->
+                <kp>10000000.0</kp>
+                <kd>1.0</kd>
+                <max_vel>1.0</max_vel>
+                <min_depth>0.001</min_depth> <!-- also influences if the base can change direction without caster does not block-->
+              </ode>
+            </contact>
+          </surface>
+      </collision>
     </gazebo>
   </xacro:macro>

File: mir_description/urdf/include/wheel.urdf.xacro (robot description, xacro)
@@ -33,10 +33,36 @@
     <!-- set the gazebo friction parameters for the wheels -->
     <gazebo reference="${prefix}${locationprefix}_wheel_link">
-      <kp value="10000000.0"/>
-      <kd value="1.0"/>
-      <mu1 value="200"/>
-      <mu2 value="200"/>
-      <maxVel>1.0</maxVel>
-      <minDepth>0.01</minDepth>
+      <!-- <mu1>1.6</mu1>
+      <mu2>1.6</mu2>
+      <min_depth>0.01</min_depth> -->
+      <collision name="${prefix}${locationprefix}_wheel_link_collision">
+        <surface>
+            <friction>
+              <ode>
+                <mu>200</mu>
+                <!-- <mu2>1.6</mu2> -->
+                <!--
+                <fdir1>0 0 1</fdir1> -->
+                <!-- <slip1>0</slip1>
+                <slip2>0</slip2> -->
+              </ode>
+              <!-- <torsional>
+                <coefficient>200</coefficient>
+                <use_patch_radius>true</use_patch_radius>
+                <surface_radius>${mir_100_act_wheel_radius}</surface_radius>
+              </torsional> -->
+            </friction>
+            <contact>
+              <ode>
+                <!-- <soft_cfm>0.0</soft_cfm>
+                <soft_erp>0.2</soft_erp> -->
+                <kp>10000000.0</kp>
+                <kd>1.0</kd>
+                <max_vel>1.0</max_vel>
+                <min_depth>0.001</min_depth>
+              </ode>
+            </contact>
+          </surface>
+      </collision>
     </gazebo>
   </xacro:macro>

Commit message: applied torsional force, updated contact collisons

File: mir_description/urdf/include/caster.urdf.xacro (robot description, xacro)
@@ -11,7 +11,4 @@
       <dynamics damping="0.5" friction="0.05"/>
     </joint>
-    <gazebo reference="${prefix}${locationprefix}_caster_rotation_joint">
-      <implicitSpringDamper>0</implicitSpringDamper>
-    </gazebo>
     <gazebo>
       <plugin name="${locationprefix}_caster_rotation_joint_states" filename="libgazebo_ros_joint_state_publisher.so">
@@ -59,4 +56,5 @@
       <child link="${prefix}${locationprefix}_caster_wheel_link" />
       <axis xyz="0 1 0" />
+      <!-- <dynamics damping="0.015" friction="0.0"/> -->
     </joint>
     <gazebo>
@@ -98,13 +96,13 @@
                 <mu>1.0</mu>
                 <mu2>1.0</mu2>
-                <!--<fdir1>0 0 1</fdir1> -->
-                <!-- <slip1>0</slip1>
-                <slip2>0</slip2> -->
+                <!-- <fdir1>1 0 0</fdir1>
+                <slip1>0.0</slip1>
+                <slip2>0.0</slip2> -->
               </ode>
-              <!-- <torsional>
-                <coefficient>200</coefficient>
-                <use_patch_radius>true</use_patch_radius>
+              <torsional>
+                <coefficient>1.0</coefficient>
+                <use_patch_radius>false</use_patch_radius>
                 <surface_radius>${mir_100_caster_wheel_radius}</surface_radius>
-              </torsional> -->
+              </torsional>
             </friction>
             <contact>
@@ -112,8 +110,8 @@
                 <!-- <soft_cfm>0.0</soft_cfm>
                 <soft_erp>0.2</soft_erp> -->
-                <kp>10000000.0</kp>
-                <kd>1.0</kd>
+                <kp>100000000.0</kp>
+                <!--<kd>1.0</kd> -->
                 <max_vel>1.0</max_vel>
-                <min_depth>0.001</min_depth> <!-- also influences if the base can change direction without caster does not block-->
+                <min_depth>0.001</min_depth>
               </ode>
             </contact>

File: mir_description/urdf/include/wheel.urdf.xacro (robot description, xacro)
@@ -9,4 +9,8 @@
       <axis xyz="0 1 0" />
       <limit effort="100" velocity="20.0" />
+      <!-- <dynamics damping="0.0" friction="0.0"/> -->
+      <!-- <gazebo reference="${prefix}${locationprefix}_wheel_joint">
+        <implicitSpringDamper>1</implicitSpringDamper>
+      </gazebo> -->
     </joint>
     <link name="${prefix}${locationprefix}_wheel_link">
@@ -40,16 +44,15 @@
             <friction>
               <ode>
-                <mu>200</mu>
-                <!-- <mu2>1.6</mu2> -->
-                <!--
-                <fdir1>0 0 1</fdir1> -->
+                <mu>300</mu>
+                <mu2>300</mu2>
+                <fdir1>0 0 1</fdir1>
                 <!-- <slip1>0</slip1>
                 <slip2>0</slip2> -->
               </ode>
-              <!-- <torsional>
-                <coefficient>200</coefficient>
-                <use_patch_radius>true</use_patch_radius>
+              <torsional>
+                <coefficient>300</coefficient>
+                <use_patch_radius>false</use_patch_radius>
                 <surface_radius>${mir_100_act_wheel_radius}</surface_radius>
-              </torsional> -->
+              </torsional>
             </friction>
             <contact>
@@ -57,7 +60,7 @@
                 <!-- <soft_cfm>0.0</soft_cfm>
                 <soft_erp>0.2</soft_erp> -->
-                <kp>10000000.0</kp>
+                <!-- <kp>10000000.0</kp>
                 <kd>1.0</kd>
-                <max_vel>1.0</max_vel>
+                <max_vel>0.01</max_vel> -->
                 <min_depth>0.001</min_depth>
               </ode>

Commit message: tuned wheel frictions and contacs more

File: mir_description/urdf/include/caster.urdf.xacro (robot description, xacro)
@@ -9,5 +9,5 @@
       <child link="${prefix}${locationprefix}_caster_rotation_link" />
       <axis xyz="0 0 1" />
-      <dynamics damping="0.5" friction="0.05"/>
+      <dynamics damping="0.0" friction="0.5"/>
     </joint>
     <gazebo>
@@ -56,5 +56,4 @@
       <child link="${prefix}${locationprefix}_caster_wheel_link" />
       <axis xyz="0 1 0" />
-      <!-- <dynamics damping="0.015" friction="0.0"/> -->
     </joint>
     <gazebo>
@@ -96,13 +95,13 @@
                 <mu>1.0</mu>
                 <mu2>1.0</mu2>
-                <!-- <fdir1>1 0 0</fdir1>
+                <fdir1>0 0 1</fdir1>
                 <slip1>0.0</slip1>
-                <slip2>0.0</slip2> -->
+                <slip2>0.5</slip2>
               </ode>
-              <torsional>
+              <!-- <torsional>
                 <coefficient>1.0</coefficient>
                 <use_patch_radius>false</use_patch_radius>
                 <surface_radius>${mir_100_caster_wheel_radius}</surface_radius>
-              </torsional>
+              </torsional> -->
             </friction>
             <contact>
@@ -112,6 +111,6 @@
                 <kp>100000000.0</kp>
                 <!--<kd>1.0</kd> -->
-                <max_vel>1.0</max_vel>
-                <min_depth>0.001</min_depth>
+                <!-- <max_vel>1.0</max_vel> -->
+                <min_depth>0.0</min_depth>
               </ode>
             </contact>

File: mir_description/urdf/include/wheel.urdf.xacro (robot description, xacro)
@@ -44,6 +44,6 @@
             <friction>
               <ode>
-                <mu>300</mu>
-                <mu2>300</mu2>
+                <mu>300.0</mu>
+                <mu2>300.0</mu2>
                 <fdir1>0 0 1</fdir1>
                 <!-- <slip1>0</slip1>
@@ -63,5 +63,5 @@
                 <kd>1.0</kd>
                 <max_vel>0.01</max_vel> -->
-                <min_depth>0.001</min_depth>
+                <min_depth>0.001</min_depth> <!-- depth needed to have contact friction-->
               </ode>
             </contact>
